File: DB25/gbscsi2.kicad_pcb (KiCad board)
At the start: 4 copper layers, 53.1 x 44.2 mm, 97 parts, among them J2 TF003, J6 DB25_Plug, SW1 SW_DIP_x02, U1 Pico W, U2 74LVT245, U3 74LVT245, U4 74AHCT1G125, U5 74LVT125, U6 74LVT125, U8 AP62250WU

Commit message: Changed diodes in BoM, minor corrections to PCB, documentation
Parts:
- removed REF**: OSHW-Logo2_9.8x8mm_SilkScreen, Symbol:OSHW-Logo2_9.8x8mm_SilkScreen
