File: DB25/gbscsi2.kicad_sch (KiCad schematic)
At the start: 104 parts, among them J2 TF003, J6 DB25_Plug, SW1 SW_DIP_x02, U4 74AHCT1G125, U8 AP62250WU

Commit message: Changed diodes in BoM, minor corrections to PCB, documentation
Parts:
- D? (x3): LCSC C8598 -> C82544
Changed lines of the file:
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@@
       (effects (font (size 1.27 1.27)))
     )
-    (property "LCSC" "C8598" (at 166.37 27.94 0)
+    (property "LCSC" "C82544" (at 166.37 27.94 0)
       (effects (font (size 1.27 1.27)) hide)
     )
@@
       (effects (font (size 1.27 1.27)))
     )
-    (property "LCSC" "C8598" (at 158.75 35.56 0)
+    (property "LCSC" "C82544" (at 158.75 35.56 0)
       (effects (font (size 1.27 1.27)) hide)
     )
@@
       (effects (font (size 1.27 1.27)))
     )
-    (property "LCSC" "C8598" (at 166.37 57.15 0)
-      (effects (font (size 1.27 1.27)) hide)
-    )
+    (property "LCSC" "C82544" (at 166.37 57.15 0)
+      (effects (font (size 1.27 1.27)) hide)
+    )

Commit message: Cleaning up, updating docs
Parts:
- C1: value 100nF -> 10uF; LCSC C14663 -> C96446
- C? (x13): symbol zuluscsi-rescue:C_Small -> Device:C_Small
- D? (x3): symbol zuluscsi-rescue:D_Schottky -> Device:D_Schottky
- R? (x59): symbol zuluscsi-rescue:R -> Device:R
Connections:
- net +3V3 renamed +3.3V
