File: rp2350_wide/gbscsi2.kicad_sch (KiCad schematic)
At the start: 180 parts, among them J1 USB_DATA, J2 TF003, J3 Conn_01x02, J4 MnL, J5 HD68, J7 Conn_01x04, Q1 AO3401A, Q10 AO3401A, Q11 AO3401A, Q12 AO3401A, Q13 AO3401A, Q14 AO3401A, Q15 AO3401A, Q16 AO3401A, Q17 AO3401A, Q18 AO3401A, Q19 AO3401A, Q2 AO3401A, Q20 AO3401A, Q21 AO3401A, Q22 AO3401A, Q23 AO3401A, Q24 AO3401A, Q25 AO3401A, Q26 AO3401A, Q27 AO3401A, Q3 AO3401A, Q4 AO3401A, Q5 AO3401A, Q6 AO3401A, Q7 AO3401A, Q8 AO3401A, Q9 AO3401A, SW1 SW_DIP_x04, U1 RP2350_80QFN, U2 W25Q128JVS, U7 AZ1117-2.85, U8 AP62250WU, U9 USB TVS, Y1 12MHz

Commit message: Redoing Wide variant - WIP
Parts:
- removed C19: 4.7nF, Capacitor_SMD:C_0402_1005Metric, symbol Device:C_Small
- removed D6: YELLOW, LED_SMD:LED_0603_1608Metric, symbol Device:LED_Small_Filled
- removed R52: 510, Resistor_SMD:R_0603_1608Metric, symbol Device:R
- removed R?: 1M, Resistor_SMD:R_0402_1005Metric, symbol Device:R
- removed R?: 4k7, Resistor_SMD:R_0603_1608Metric, symbol Device:R
- removed R?: 1k, Resistor_SMD:R_0603_1608Metric, symbol Device:R
- removed U?: 74LVT125, Package_SO:TSSOP-14_4.4x5mm_P0.65mm, symbol 74xx:74LVC125
- added J6: Conn_01x05, Connector_PinHeader_2.54mm:PinHeader_1x05_P2.54mm_Vertical, symbol Connector_Generic:Conn_01x05
- added J8: Conn_01x02, Connector_PinHeader_2.54mm:PinHeader_1x02_P2.54mm_Vertical, symbol Connector_Generic:Conn_01x02
- added R3: 27, Resistor_SMD:R_0402_1005Metric, symbol Device:R
- added R? (x4): 4k7, Resistor_SMD:R_0603_1608Metric, symbol Device:R
- added SW2: GT-TC108A-H034-L1S, symbol Switch:SW_SPST
- added U?: 74LVT125, Package_SO:TSSOP-14_4.4x5mm_P0.65mm, symbol 74xx:74LVC125
- C26, C35: footprint Capacitor_SMD:C_0402_1005Metric -> Capacitor_SMD:C_0603_1608Metric; LCSC C23733 -> C19666; LCSC Part # C23733 -> C19666
- C36: value 100n -> 4.7uF; LCSC C307331 -> C23733; LCSC Part # C307331 -> C23733
Connections:
- net MCU_RST is gone; now on net ~{MCU_SDP1}: U1.21 (GPIO21)
- net +3V3: now also J6.1 (Pin_1), R3.2, R?.1, R?.2, R?.2, R?.2; no longer C36.1, R?.1, U1.54 (GPIO43_ADC3), U1.55 (GPIO44_ADC4), U1.61 (VREG_AVDD)
- net GND: now also J1.S1 (SHIELD), R?.1, J6.4 (Pin_4), J8.1 (Pin_1), SW2.2 (B); no longer U?.9
- net SDIO_CLK: now also U1.43 (GPIO34); no longer U1.8 (GPIO10)
- net SDIO_CMD: now also U1.44 (GPIO35); no longer U1.9 (GPIO11)
- net SDIO_D0: now also U1.45 (GPIO36); no longer U1.11 (GPIO12)
- net SDIO_D1: now also U1.46 (GPIO37); no longer U1.12 (GPIO13)
- net SDIO_D2: now also U1.47 (GPIO38); no longer U1.13 (GPIO14)
- net SDIO_D3: now also U1.48 (GPIO39); no longer U1.14 (GPIO15)
- net ~{BUS_DIR}: now also U?.8; no longer R?.2, U1.7 (GPIO9)
- net ~{DEBUG}: now also R?.2, U1.40 (GPIO32); no longer R?.1, R?.2, SW1.7
- net ~{MCU_ACK}: now also R?.2
- net ~{MCU_ATTN}: now also U1.26 (GPIO25); no longer R?.2, U1.37 (GPIO29)
- net ~{MCU_BSY_OUT}: now also U1.78 (GPIO1); no longer U1.36 (GPIO28)
- net ~{MCU_CD/SEL_IN}: now also U1.25 (GPIO24); no longer U1.18 (GPIO18)
- net ~{MCU_IO}: now also U1.36 (GPIO28); no longer R?.2, U1.22 (GPIO22)
- net ~{MCU_MSG/BSY_IN}: now also U1.27 (GPIO26); no longer U1.20 (GPIO20)
- net ~{MCU_REQ}: now also R?.2, U1.22 (GPIO22); no longer R?.2, U1.17 (GPIO17)
- net ~{MCU_SD0}: now also U1.1 (GPIO4); no longer U1.77 (GPIO0)
- net ~{MCU_SD10}: now also U1.13 (GPIO14); no longer U1.40 (GPIO32)
- net ~{MCU_SD11}: now also U1.14 (GPIO15); no longer U1.42 (GPIO33)
- net ~{MCU_SD12}: now also U1.16 (GPIO16); no longer U1.43 (GPIO34)
- net ~{MCU_SD13}: now also U1.17 (GPIO17); no longer U1.44 (GPIO35)
- net ~{MCU_SD14}: now also U1.18 (GPIO18); no longer U1.45 (GPIO36)
- net ~{MCU_SD15}: now also U1.19 (GPIO19); no longer U1.46 (GPIO37)
- net ~{MCU_SD1}: now also U1.2 (GPIO5); no longer U1.78 (GPIO1)
- net ~{MCU_SD2}: now also U1.3 (GPIO6); no longer U1.79 (GPIO2)
- net ~{MCU_SD3}: now also U1.4 (GPIO7); no longer U1.80 (GPIO3)
- net ~{MCU_SD4}: now also U1.6 (GPIO8); no longer U1.1 (GPIO4)
- net ~{MCU_SD5}: now also U1.7 (GPIO9); no longer U1.2 (GPIO5)
- net ~{MCU_SD6}: now also U1.8 (GPIO10); no longer U1.3 (GPIO6)
- net ~{MCU_SD7}: now also U1.9 (GPIO11); no longer U1.4 (GPIO7)
- net ~{MCU_SD8}: now also U1.11 (GPIO12); no longer U1.38 (GPIO30)
- net ~{MCU_SD9}: now also U1.12 (GPIO13); no longer U1.39 (GPIO31)
- net ~{MCU_SDP1}: no longer U1.47 (GPIO38)
- net ~{MCU_SDP}: now also U1.20 (GPIO20); no longer U1.6 (GPIO8)
- net ~{MCU_SEL_OUT}: now also U1.77 (GPIO0); no longer U1.19 (GPIO19)
- net ~{MCU_RST_IN}: now reaches U?.11
- net ~{MCU_RST_IN}: now also U1.79 (GPIO2)
- net BUS_DIR: now reaches U1.23 (GPIO23)
- net BUS_DIR: now also R?.2, U?.9
- net GPIO16: no longer names the net of D1.2 (A), J3.1 (Pin_1)
- net GPIO16: now also U1.42 (GPIO33); no longer U1.16 (GPIO16)
- net ~{RST_OUT} renamed ~{MCU_RST_OUT}
- net ~{MCU_RST_OUT}: now also U1.80 (GPIO3)
- new net: R?.1, R?.2, SW1.7
- new net: C36.1, R3.1, U1.61 (VREG_AVDD)
- new net EJECT: J8.2 (Pin_2), R?.2, SW2.1 (A), U1.55 (GPIO44_ADC4)
- new net I²C_INT: J6.5 (Pin_5), R?.1, U1.39 (GPIO31)
- new net I²C_SCL: J6.3 (Pin_3), R?.1, U1.38 (GPIO30)
- new net I²C_SDA: J6.2 (Pin_2), R?.1, U1.37 (GPIO29)
- no-connect marks 18 -> 14
Other:
- note added: "Ideally 2.2k but whatever"
- note added: "Make sure R48 and R49 are close to RP2350"
- note added: "Meets revised Pi VREG guidelines"
- note added: "USB-C Spec §3.2.1¶11"
- note removed: "Make sure R3 and R4 are close to RP2350"
- note removed: "PD as per ZS 2023d"
- title: GBSCSI 2 -> GBSCSI 2 Wide
- moved on the sheet: C?, J7, R?, U?C, U?E
