File: 2.5_to_3.5_SCA_carrier_untested/SCA.kicad_sch (KiCad schematic)
At the start: 11 parts, among them J1 SCSI_50-2P_2mm, J2 Conn_02x40_Counter_Clockwise

Commit message: Cleaning up, updating docs
Connections:
- net TERMPWR: no longer names the net of J1.24 (Pin_24)
- no-connect marks 32 -> 35
Changed lines of the file:
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@@
   (no_connect (at 39.37 29.21))
   (no_connect (at 97.79 29.21))
+  (no_connect (at 110.49 29.21))
   (no_connect (at 97.79 26.67))
   (no_connect (at 97.79 31.75))
@@
   (no_connect (at 97.79 95.25))
   (no_connect (at 97.79 100.33))
+  (no_connect (at 110.49 113.03))
+  (no_connect (at 52.07 67.31))
   (no_connect (at 97.79 44.45))
   (no_connect (at 97.79 102.87))
@@
     (stroke (width 0) (type default))
   )
-  (wire (pts (xy 52.07 67.31) (xy 55.88 67.31))
-    (stroke (width 0) (type default))
-  )
   (wire (pts (xy 118.11 34.29) (xy 118.11 39.37))
     (stroke (width 0) (type default))
@@
     (effects (font (size 1.27 1.27)) (justify left bottom))
   )
-  (label "TERMPWR" (at 55.88 67.31 0) (fields_autoplaced)
-    (effects (font (size 1.27 1.27)) (justify left bottom))
-  )
