File: 3.5/gbscsi2.kicad_sch (KiCad schematic)
At the start: 120 parts, among them J1 Conn_01x02, J2 TF003, J3 Conn_01x04, J4 Conn_01x04, J6 SCSI_50P_2.54mm, Q1 AO3401A, Q10 AO3401A, Q11 AO3401A, Q12 AO3401A, Q13 AO3401A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

Commit message: Changed diodes in BoM, minor corrections to PCB, documentation
Parts:
- D? (x4): LCSC C8598 -> C82544
Changed lines of the file:
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@@
       (effects (font (size 1.27 1.27)))
     )
-    (property "LCSC" "C8598" (at 200.66 27.94 0)
+    (property "LCSC" "C82544" (at 200.66 27.94 0)
       (effects (font (size 1.27 1.27)) hide)
     )
@@
       (effects (font (size 1.27 1.27)))
     )
-    (property "LCSC" "C8598" (at 193.04 35.56 0)
+    (property "LCSC" "C82544" (at 193.04 35.56 0)
       (effects (font (size 1.27 1.27)) hide)
     )
@@
       (effects (font (size 1.27 1.27)))
     )
-    (property "LCSC" "C8598" (at 200.66 57.15 0)
+    (property "LCSC" "C82544" (at 200.66 57.15 0)
       (effects (font (size 1.27 1.27)) hide)
     )
@@
       (effects (font (size 1.27 1.27)))
     )
-    (property "LCSC" "C8598" (at 200.66 66.04 0)
+    (property "LCSC" "C82544" (at 200.66 66.04 0)
       (effects (font (size 1.27 1.27)) hide)
     )

Commit message: Cleaning up, updating docs
Parts:
- C1: value 100nF -> 10uF; LCSC C14663 -> C96446
- C? (x17): symbol zuluscsi-rescue:C_Small -> Device:C_Small
- D? (x4): symbol zuluscsi-rescue:D_Schottky -> Device:D_Schottky
- R? (x24): symbol zuluscsi-rescue:R -> Device:R
Connections:
- net +3V3 renamed +3.3V
