File: rp2350_2.5_3.5_narrow/gbscsi2.kicad_pcb (KiCad board)
At the start: 4 copper layers, 69.5 x 93.5 mm, 147 parts, among them J1 USB_DATA, J2 TF003, J3 Conn_01x02, J4 Conn_01x04, J5 SCSI_50-2P_2mm, J6 SCSI_50P_2.54mm, J7 Conn_01x04, Q1 AO3401A, Q10 AO3401A, Q11 AO3401A, Q12 AO3401A, Q13 AO3401A, Q14 AO3401A, Q15 AO3401A, Q16 AO3401A, Q17 AO3401A, Q18 AO3401A, Q2 AO3401A, Q3 AO3401A, Q4 AO3401A, Q5 AO3401A, Q6 AO3401A, Q7 AO3401A, Q8 AO3401A, Q9 AO3401A, SW1 SW_DIP_x04, U1 RP2350_60QFN, U10 W25Q128JVS, U2 74LVT245, U3 74LVT245, U4 74AHCT1G125, U5 74LVT125, U6 74LVT125, U7 AZ1117-2.85, U8 AP62250WU, U9 USB TVS, Y1 12MHz

Commit message: Re-sorting things around
Parts:
- removed C19: 4.7nF, Capacitor_SMD:C_0402_1005Metric
- removed R15: 1M, Resistor_SMD:R_0402_1005Metric
Connections:
- J1 pad S1: Net-(J1-SHIELD) -> GND
Routing:
- net Net-(J1-SHIELD): track 23.1 -> 0.00 mm
Other:
- board text added: "(c)2024, 2025 grm"
- board text added: "pcb v1.1"
- board text removed: "(c)2024 grm"
- board text removed: "pcb v1.0"

Commit message: Cleaning up, updating docs
Parts:
- C1: value 100nF -> 10uF
Changed lines of the file:
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@@
     (descr "Capacitor SMD 0603 (1608 Metric), square (rectangular) end terminal, IPC_7351 nominal, (Body size source: IPC-SM-782 page 76, https://www.pcb-3d.com/wordpress/wp-content/uploads/ipc-sm-782a_amendment_1_and_2.pdf), generated with kicad-footprint-generator")
     (tags "capacitor")
-    (property "LCSC" "C14663")
-    (property "LCSC Part #" "C14663")
+    (property "LCSC" "C96446")
+    (property "LCSC Part #" "C96446")
     (property "Sheetfile" "gbscsi2.kicad_sch")
     (property "Sheetname" "")
@@
         (effects (font (size 1 1) (thickness 0.15)))
     )
-    (fp_text value "100nF" (at 0 1.43 -270) (layer "F.Fab")
+    (fp_text value "10uF" (at 0 1.43 -270) (layer "F.Fab")
         (effects (font (size 1 1) (thickness 0.15)))
     )
