File: rp2350_2.5_3.5_narrow/gbscsi2.kicad_sch (KiCad schematic)
At the start: 154 parts, among them J1 USB_DATA, J2 TF003, J3 Conn_01x02, J4 Conn_01x04, J5 SCSI_50-2P_2mm, J6 SCSI_50P_2.54mm, J7 Conn_01x04, Q1 AO3401A, Q10 AO3401A, Q11 AO3401A, Q12 AO3401A, Q13 AO3401A, Q14 AO3401A, Q15 AO3401A, Q16 AO3401A, Q17 AO3401A, Q18 AO3401A, Q2 AO3401A, Q3 AO3401A, Q4 AO3401A, Q5 AO3401A, Q6 AO3401A, Q7 AO3401A, Q8 AO3401A, Q9 AO3401A, SW1 SW_DIP_x04, U1 RP2350_60QFN, U2 W25Q128JVS, U4 74AHCT1G125, U7 AZ1117-2.85, U8 AP62250WU, U9 USB TVS, Y1 12MHz

Commit message: Re-sorting things around
Parts:
- removed C19: 4.7nF, Capacitor_SMD:C_0402_1005Metric, symbol Device:C_Small
- removed R?: 1M, Resistor_SMD:R_0402_1005Metric, symbol zuluscsi-rescue:R
Connections:
- net GND: now also J1.S1 (SHIELD)
Changed lines of the file:
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@@
   (junction (at 472.44 182.88) (diameter 0) (color 0 0 0 0)
   )
-  (junction (at 55.88 257.81) (diameter 0) (color 0 0 0 0)
-  )
   (junction (at 481.33 69.85) (diameter 0) (color 0 0 0 0)
   )
@@
   (junction (at 55.88 215.9) (diameter 0) (color 0 0 0 0)
   )
-  (junction (at 66.04 265.43) (diameter 0.9144) (color 0 0 0 0)
-  )
   (junction (at 130.81 161.29) (diameter 0) (color 0 0 0 0)
   )
@@
   (junction (at 271.78 165.1) (diameter 0) (color 0 0 0 0)
   )
+  (junction (at 66.04 257.81) (diameter 0) (color 0 0 0 0)
+  )
   (junction (at 472.44 77.47) (diameter 0) (color 0 0 0 0)
   )
@@
   (junction (at 121.92 27.94) (diameter 0) (color 0 0 0 0)
   )
-  (junction (at 59.69 265.43) (diameter 0) (color 0 0 0 0)
-  )
   (junction (at 168.91 93.98) (diameter 0) (color 0 0 0 0)
   )
@@
     (stroke (width 0) (type default))
   )
-  (wire (pts (xy 55.88 265.43) (xy 59.69 265.43))
-    (stroke (width 0) (type solid))
-  )
   (wire (pts (xy 116.84 186.69) (xy 111.76 186.69))
     (stroke (width 0) (type default))
@@
     (stroke (width 0) (type default))
   )
-  (wire (pts (xy 66.04 254) (xy 66.04 265.43))
+  (wire (pts (xy 66.04 254) (xy 66.04 257.81))
     (stroke (width 0) (type solid))
   )
@@
     (stroke (width 0) (type default))
   )
-  (wire (pts (xy 59.69 265.43) (xy 66.04 265.43))
+  (wire (pts (xy 55.88 257.81) (xy 66.04 257.81))
     (stroke (width 0) (type solid))
   )
@@
     (stroke (width 0) (type default))
   )
-  (wire (pts (xy 66.04 265.43) (xy 66.04 266.7))
+  (wire (pts (xy 66.04 257.81) (xy 66.04 266.7))
     (stroke (width 0) (type solid))
   )
@@
     (stroke (width 0) (type default))
   )
-  (wire (pts (xy 59.69 257.81) (xy 59.69 259.08))
-    (stroke (width 0) (type solid))
-  )
   (wire (pts (xy 185.42 125.73) (xy 185.42 127))
     (stroke (width 0) (type default))
@@
     (stroke (width 0) (type default))
   )
-  (wire (pts (xy 59.69 264.16) (xy 59.69 265.43))
-    (stroke (width 0) (type solid))
-  )
   (wire (pts (xy 148.59 121.92) (xy 148.59 127))
     (stroke (width 0) (type default))
@@
     (stroke (width 0) (type default))
   )
-  (wire (pts (xy 55.88 257.81) (xy 59.69 257.81))
-    (stroke (width 0) (type solid))
-  )
   (wire (pts (xy 497.84 64.77) (xy 494.03 64.77))
     (stroke (width 0) (type default))
@@
     )
   )
-  (symbol (lib_id "zuluscsi-rescue:R") (at 55.88 261.62 0) (mirror y) (unit 1)
-    (in_bom yes) (on_board yes) (dnp no)
-    (property "Reference" "R?" (at 53.34 261.62 90)
-      (effects (font (size 1.27 1.27)))
-    )
-    (property "Value" "1M" (at 55.88 261.62 90)
-      (effects (font (size 1.27 1.27)))
-    )
-    (property "Footprint" "Resistor_SMD:R_0402_1005Metric" (at 57.658 261.62 90)
-      (effects (font (size 1.27 1.27)) hide)
-    )
-    (property "Datasheet" "" (at 55.88 261.62 0)
-      (effects (font (size 1.27 1.27)))
-    )
-    (property "LCSC" "C26083" (at 55.88 261.62 0)
-      (effects (font (size 1.27 1.27)) hide)
-    )
-    (property "LCSC Part #" "C26083" (at 55.88 261.62 0)
-      (effects (font (size 1.27 1.27)) hide)
-    )
-    (pin "1")
-    (pin "2")
-    (instances
-      (project "ZuluSCSI-Pico-OSHW"
-        (path "/0a1a4d88-972a-46ce-b25e-6cb796bd41f7/00000000-0000-0000-0000-000055ff7cc4"
-          (reference "R?") (unit 1)
-        )
-      )
-      (project "cpu"
-        (path "/45b7fe01-a2fa-40c2-a3a2-4a9ae7c34dba"
-          (reference "R?") (unit 1)
-        )
-      )
-      (project "gbscsi2"
-        (path "/81c2a5db-c508-405c-87d7-d49be9ddd5e4"
-          (reference "R15") (unit 1)
-        )
-      )
-    )
-  )
   (symbol (lib_id "Device:C") (at 71.12 29.21 0) (unit 1)
     (in_bom yes) (on_board yes) (dnp no)
@@
         )
       )
-    )
-  )
-  (symbol (lib_id "Device:C_Small") (at 59.69 261.62 0) (mirror y) (unit 1)
-    (in_bom yes) (on_board yes) (dnp no)
-    (property "Reference" "C19" (at 63.5 259.08 0)
-      (effects (font (size 1.27 1.27)) (justify left))
-    )
-    (property "Value" "4.7nF" (at 66.04 264.16 0)
-      (effects (font (size 1.27 1.27)) (justify left))
-    )
-    (property "Footprint" "Capacitor_SMD:C_0402_1005Metric" (at 59.69 261.62 0)
-      (effects (font (size 1.27 1.27)) hide)
-    )
-    (property "Datasheet" "~" (at 59.69 261.62 0)
-      (effects (font (size 1.27 1.27)) hide)
-    )
-    (property "LCSC" "C346200" (at 59.69 261.62 0)
-      (effects (font (size 1.27 1.27)) hide)
-    )
-    (property "LCSC Part #" "C346200" (at 59.69 261.62 0)
-      (effects (font (size 1.27 1.27)) hide)
-    )
-    (pin "1")
-    (pin "2")
-    (instances
-      (project "gbscsi2"
-        (path "/81c2a5db-c508-405c-87d7-d49be9ddd5e4"
-          (reference "C19") (unit 1)
-        )
-      )
-      (project "poe_hat_v1.4.2"
-        (path "/84fe1d92-0d61-4eda-acb4-e2fc63573041"
-          (reference "C8") (unit 1)
-        )
-      )

Commit message: Cleaning up, updating docs
Parts:
- C1: value 100nF -> 10uF; LCSC C14663 -> C96446; LCSC Part # C14663 -> C96446
- C? (x17): symbol zuluscsi-rescue:C_Small -> Device:C_Small
- D? (x4): symbol zuluscsi-rescue:D_Schottky -> Device:D_Schottky
- R? (x27): symbol zuluscsi-rescue:R -> Device:R
Connections:
- net +3V3: no longer C1.1, C?.1, C?.1, C?.1, C?.1, C?.1, C?.1, C?.1, C?.1, J2.4 (VDD), J7.1 (Pin_1), L2.2, R?.1, R?.1, R?.1, R?.1, R?.1, R?.1, R?.1, R?.2, R?.2, R?.2, R?.2, R?.2, R?.2, U4.5 (VCC), U?.14 (VCC), U?.14 (VCC), U?.20 (VCC), U?.20 (VCC)
- new net +3.3V: C1.1, C?.1, C?.1, C?.1, C?.1, C?.1, C?.1, C?.1, C?.1, J2.4 (VDD), J7.1 (Pin_1), L2.2, R?.1, R?.1, R?.1, R?.1, R?.1, R?.1, R?.1, R?.2, R?.2, R?.2, R?.2, R?.2, R?.2, U4.5 (VCC), U?.14 (VCC), U?.14 (VCC), U?.20 (VCC), U?.20 (VCC)

Commit message: Minor BoM fixes, added left-behind HD68 variant eject switch
Parts:
- U1: LCSC C9900136995 -> C42411118; LCSC Part # C9900136995 -> C42411118
Changed lines of the file:
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@@
       (effects (font (size 1.27 1.27)) hide)
     )
-    (property "LCSC Part #" "C9900136995" (at 115.57 78.74 0)
+    (property "LCSC Part #" "C42411118" (at 115.57 78.74 0)
       (effects (font (size 1.27 1.27)) hide)
     )
-    (property "LCSC" "C9900136995" (at 115.57 78.74 0)
+    (property "LCSC" "C42411118" (at 115.57 78.74 0)
       (effects (font (size 1.27 1.27)) hide)
     )
