File: rp2350_HD68_3.5/gbscsi2.kicad_pcb (KiCad board)
At the start: 4 copper layers, 100 x 93.5 mm, 170 parts, among them J1 USB_DATA, J2 TF003, J3 Conn_01x02, J4 MnL, J5 HD68, J6 Conn_01x05, J7 Conn_01x04, J8 Conn_01x02, Q1 AO3401A, Q10 AO3401A, Q11 AO3401A, Q12 AO3401A, Q13 AO3401A, Q14 AO3401A, Q15 AO3401A, Q16 AO3401A, Q17 AO3401A, Q18 AO3401A, Q19 AO3401A, Q2 AO3401A, Q20 AO3401A, Q21 AO3401A, Q22 AO3401A, Q23 AO3401A, Q24 AO3401A, Q25 AO3401A, Q26 AO3401A, Q27 AO3401A, Q3 AO3401A, Q4 AO3401A, Q5 AO3401A, Q6 AO3401A, Q7 AO3401A, Q8 AO3401A, Q9 AO3401A, SW1 SW_DIP_x04, U1 RP2350_80QFN, U10 W25Q128JVS, U11 74LVT245, U2 74LVT245, U3 74LVT245, U4 74LVT125, U5 74LVT125, U6 74LVT125, U7 AZ1117-2.85, U8 AP62250WU, U9 USB TVS, Y1 12MHz

Commit message: Re-sorting things around
Other:
- board text added: "2350W"
- board text added: "artwork © grm, 2025 github.com/GeorgeRudolf/GBSCSI2"
- board text removed: "artwork © grm, 2024 github.com/GeorgeRudolf/GBSCSI2"

Commit message: Cleaning up, updating docs
Parts:
- C1: value 100nF -> 10uF
Changed lines of the file:
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@@
     (descr "Capacitor SMD 0603 (1608 Metric), square (rectangular) end terminal, IPC_7351 nominal, (Body size source: IPC-SM-782 page 76, https://www.pcb-3d.com/wordpress/wp-content/uploads/ipc-sm-782a_amendment_1_and_2.pdf), generated with kicad-footprint-generator")
     (tags "capacitor")
-    (property "LCSC" "C14663")
-    (property "LCSC Part #" "C14663")
+    (property "LCSC" "C96446")
+    (property "LCSC Part #" "C96446")
     (property "Sheetfile" "gbscsi2.kicad_sch")
     (property "Sheetname" "")
@@
         (effects (font (size 1 1) (thickness 0.15)))
     )
-    (fp_text value "100nF" (at 0 1.43 -270) (layer "F.Fab")
+    (fp_text value "10uF" (at 0 1.43 -270) (layer "F.Fab")
         (effects (font (size 1 1) (thickness 0.15)))
     )
