File: rp2350_HD68_3.5/gbscsi2.kicad_sch (KiCad schematic)
At the start: 182 parts, among them J1 USB_DATA, J2 TF003, J3 Conn_01x02, J4 MnL, J5 HD68, J6 Conn_01x05, J7 Conn_01x04, J8 Conn_01x02, Q1 AO3401A, Q10 AO3401A, Q11 AO3401A, Q12 AO3401A, Q13 AO3401A, Q14 AO3401A, Q15 AO3401A, Q16 AO3401A, Q17 AO3401A, Q18 AO3401A, Q19 AO3401A, Q2 AO3401A, Q20 AO3401A, Q21 AO3401A, Q22 AO3401A, Q23 AO3401A, Q24 AO3401A, Q25 AO3401A, Q26 AO3401A, Q27 AO3401A, Q3 AO3401A, Q4 AO3401A, Q5 AO3401A, Q6 AO3401A, Q7 AO3401A, Q8 AO3401A, Q9 AO3401A, SW1 SW_DIP_x04, SW2 GT-TC108A-H034-L1S, U1 RP2350_80QFN, U2 W25Q128JVS, U7 AZ1117-2.85, U8 AP62250WU, U9 USB TVS, Y1 12MHz

Commit message: Cleaning up, updating docs
Parts:
- C1: value 100nF -> 10uF; LCSC C14663 -> C96446; LCSC Part # C14663 -> C96446
Changed lines of the file:
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@@
       (effects (font (size 1.27 1.27)))
     )
-    (property "Value" "100nF" (at 82.55 217.17 0)
+    (property "Value" "10uF" (at 82.55 217.17 0)
       (effects (font (size 1.27 1.27)))
     )
@@
       (effects (font (size 1.27 1.27)) hide)
     )
-    (property "LCSC" "C14663" (at 87.63 215.9 0)
+    (property "LCSC" "C96446" (at 87.63 215.9 0)
       (effects (font (size 1.27 1.27)) hide)
     )
-    (property "LCSC Part #" "C14663" (at 87.63 215.9 0)
+    (property "LCSC Part #" "C96446" (at 87.63 215.9 0)
       (effects (font (size 1.27 1.27)) hide)
     )

Commit message: Minor BoM fixes, added left-behind HD68 variant eject switch
Parts:
- SW2: footprint (none) -> GBSCSI:SW_Push_1P1T-MP_NO_Horizontal_Alps_SKRTLAE010
- U1: LCSC C9900136995 -> C42415655; LCSC Part # C9900136995 -> C42415655
Changed lines of the file:
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@@
       (effects (font (size 1.27 1.27)))
     )
-    (property "Footprint" "" (at 170.18 161.29 0)
+    (property "Footprint" "GBSCSI:SW_Push_1P1T-MP_NO_Horizontal_Alps_SKRTLAE010" (at 170.18 161.29 0)
       (effects (font (size 1.27 1.27)) hide)
     )
@@
       (effects (font (size 1.27 1.27)) hide)
     )
-    (property "LCSC Part #" "C9900136995" (at 115.57 78.74 0)
+    (property "LCSC Part #" "C42415655" (at 115.57 78.74 0)
       (effects (font (size 1.27 1.27)) hide)
     )
-    (property "LCSC" "C9900136995" (at 115.57 78.74 0)
+    (property "LCSC" "C42415655" (at 115.57 78.74 0)
       (effects (font (size 1.27 1.27)) hide)
     )
