File: rp2350_SCA_2.5/gbscsi2.kicad_pcb (KiCad board)
At the start: 4 copper layers, 69.5 x 93.6 mm, 105 parts, among them J1 USB_DATA, J2 TF003, J3 Conn_01x02, J6 Conn_01x05, J7 Conn_01x04, J8 Conn_01x02, J9 Conn_02x40_Counter_Clockwise, SW1 SW_DIP_x03, U1 RP2350_80QFN, U10 W25Q128JVS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

Commit message: Attempting to organize sheet details, adding eject buttons to Wide variants
Parts:
- added SW2: GT-TC108A-H034-L1S, GBSCSI:SW_Push_1P1T-MP_NO_Horizontal_Alps_SKRTLAE010, F.Cu at (49.0, 116.9)
- moved R66 3.45 mm to (49.4, 108.3)
- moved J8 3.45 mm to (47.5, 111.4)
Routing:
- net /EJECT: track 27.7 -> 39.8 mm
Other:
- board text added: "Eject"

Commit message: Cleaning up, updating docs
Parts:
- C1: value 100nF -> 10uF
Changed lines of the file:
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@@
     (descr "Capacitor SMD 0603 (1608 Metric), square (rectangular) end terminal, IPC_7351 nominal, (Body size source: IPC-SM-782 page 76, https://www.pcb-3d.com/wordpress/wp-content/uploads/ipc-sm-782a_amendment_1_and_2.pdf), generated with kicad-footprint-generator")
     (tags "capacitor")
-    (property "LCSC" "C14663")
-    (property "LCSC Part #" "C14663")
+    (property "LCSC" "C96446")
+    (property "LCSC Part #" "C96446")
     (property "Sheetfile" "gbscsi2.kicad_sch")
     (property "Sheetname" "")
@@
         (effects (font (size 1 1) (thickness 0.15)))
     )
-    (fp_text value "100nF" (at 0 1.43 -270) (layer "F.Fab")
+    (fp_text value "10uF" (at 0 1.43 -270) (layer "F.Fab")
         (effects (font (size 1 1) (thickness 0.15)))
     )
