File: rp2350_SCA_2.5/gbscsi2.kicad_sch (KiCad schematic)
At the start: 117 parts, among them J1 USB_DATA, J2 TF003, J3 Conn_01x02, J6 Conn_01x05, J7 Conn_01x04, J8 Conn_01x02, J9 Conn_02x40_Counter_Clockwise, SW1 SW_DIP_x03, SW2 GT-TC108A-H034-L1S, U1 RP2350_80QFN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

Commit message: Re-sorting things around
Parts:
- SW1: footprint Button_Switch_SMD:SW_DIP_SPSTx04_Slide_6.7x11.72mm_W8.61mm_P2.54mm_LowProfile -> Button_Switch_SMD:SW_DIP_SPSTx03_Slide_6.7x9.18mm_W8.61mm_P2.54mm_LowProfile; LCSC C5160841 -> C2842910; LCSC Part # C5160841 -> C2842910
Changed lines of the file:
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@@
       (effects (font (size 1.27 1.27)))
     )
-    (property "Footprint" "Button_Switch_SMD:SW_DIP_SPSTx04_Slide_6.7x11.72mm_W8.61mm_P2.54mm_LowProfile" (at 172.72 209.55 0)
+    (property "Footprint" "Button_Switch_SMD:SW_DIP_SPSTx03_Slide_6.7x9.18mm_W8.61mm_P2.54mm_LowProfile" (at 172.72 209.55 0)
       (effects (font (size 1.27 1.27)) hide)
     )
@@
       (effects (font (size 1.27 1.27)) hide)
     )
-    (property "LCSC" "C5160841" (at 172.72 209.55 0)
+    (property "LCSC" "C2842910" (at 172.72 209.55 0)
       (effects (font (size 1.27 1.27)) hide)
     )
-    (property "LCSC Part #" "C5160841" (at 172.72 209.55 0)
+    (property "LCSC Part #" "C2842910" (at 172.72 209.55 0)
       (effects (font (size 1.27 1.27)) hide)
     )

Commit message: Attempting to organize sheet details, adding eject buttons to Wide variants
Parts:
- SW2: footprint (none) -> GBSCSI:SW_Push_1P1T-MP_NO_Horizontal_Alps_SKRTLAE010
Changed lines of the file:
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@@
   (title_block
     (title "GBSCSI 2 Wide")
-    (date "2025-03-08")
-    (rev "0.1.1")
+    (date "2025-03-09")
+    (rev "0.1")
     (comment 1 "Drawn by; George Rudolf Mezzomo")
-    (comment 2 "GBSCSI model 2, HD68W header, 3.5\" form factor compatible, discrete RP2350")
+    (comment 2 "GBSCSI model 2, SCA header, 2.5\" form factor compatible, discrete RP2350")
   )
   (junction (at 109.22 27.94) (diameter 0) (color 0 0 0 0)
@@
       (effects (font (size 1.27 1.27)))
     )
-    (property "Footprint" "" (at 170.18 161.29 0)
+    (property "Footprint" "GBSCSI:SW_Push_1P1T-MP_NO_Horizontal_Alps_SKRTLAE010" (at 170.18 161.29 0)
       (effects (font (size 1.27 1.27)) hide)
     )

Commit message: Cleaning up, updating docs
Parts:
- C1: value 100nF -> 10uF; LCSC C14663 -> C96446; LCSC Part # C14663 -> C96446
Changed lines of the file:
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@@
       (effects (font (size 1.27 1.27)))
     )
-    (property "Value" "100nF" (at 82.55 217.17 0)
+    (property "Value" "10uF" (at 82.55 217.17 0)
       (effects (font (size 1.27 1.27)))
     )
@@
       (effects (font (size 1.27 1.27)) hide)
     )
-    (property "LCSC" "C14663" (at 87.63 215.9 0)
+    (property "LCSC" "C96446" (at 87.63 215.9 0)
       (effects (font (size 1.27 1.27)) hide)
     )
-    (property "LCSC Part #" "C14663" (at 87.63 215.9 0)
+    (property "LCSC Part #" "C96446" (at 87.63 215.9 0)
       (effects (font (size 1.27 1.27)) hide)
     )

Commit message: Minor BoM fixes, added left-behind HD68 variant eject switch
Parts:
- U1: LCSC C9900136995 -> C42415655; LCSC Part # C9900136995 -> C42415655
Changed lines of the file:
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@@
       (effects (font (size 1.27 1.27)) hide)
     )
-    (property "LCSC Part #" "C9900136995" (at 115.57 78.74 0)
+    (property "LCSC Part #" "C42415655" (at 115.57 78.74 0)
       (effects (font (size 1.27 1.27)) hide)
     )
-    (property "LCSC" "C9900136995" (at 115.57 78.74 0)
+    (property "LCSC" "C42415655" (at 115.57 78.74 0)
       (effects (font (size 1.27 1.27)) hide)
     )
