File: EDA/Common Sheets/scsi_conn_SCA_TH.kicad_sch (KiCad schematic)
At the start: 3 parts, among them J1 Conn_02x40_Counter_Clockwise

Commit message: Fixing up schematics for SCA before layout
Other:
- title: GBSCSI2 Common Platform - SCSI Headers, 2mm/2.54mm -> GBSCSI2 Common Platform - SCA SCSI Connector, Thru Hole
Changed lines of the file:
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@@
 	(paper "A5" portrait)
 	(title_block
-		(title "GBSCSI2 Common Platform - SCSI Headers, 2mm/2.54mm")
+		(title "GBSCSI2 Common Platform - SCA SCSI Connector, Thru Hole")
 		(date "2026-02-01")
 		(rev "2.0")
@@
 	)
 	(junction
+		(at 100.33 144.78)
+		(diameter 0)
+		(color 0 0 0 0)
+	)
+	(junction
 		(at 100.33 63.5)
 		(diameter 0)
@@
 	(wire
 		(pts
-			(xy 100.33 146.05) (xy 100.33 139.7)
+			(xy 100.33 146.05) (xy 100.33 144.78)
 		)
 		(stroke
@@
 		(pts
 			(xy 73.66 78.74) (xy 80.01 78.74)
+		)
+		(stroke
+			(width 0)
+			(type default)
+		)
+	)
+	(wire
+		(pts
+			(xy 100.33 144.78) (xy 100.33 139.7)
 		)
 		(stroke
@@
 					(unit 1)
 				)
+			)
+		)
+	)
+	(symbol
+		(lib_id "power:PWR_FLAG")
+		(at 100.33 144.78 90)
+		(unit 1)
+		(exclude_from_sim no)
+		(in_bom yes)
+		(on_board yes)
+		(dnp no)
+		(fields_autoplaced yes)
+		(property "Reference" "#FLG07"
+			(at 98.425 144.78 0)
+			(effects
+				(font
+					(size 1.2 1.2)
+				)
+				(hide yes)
+			)
+		)
+		(property "Value" "PWR_FLAG"
+			(at 96.52 144.7799 90)
+			(effects
+				(font
+					(size 1.27 1.27)
+				)
+				(justify left)
+			)
+		)
+		(property "Footprint" ""
+			(at 100.33 144.78 0)
+			(effects
+				(font
+					(size 1.27 1.27)
+				)
+				(hide yes)
+			)
+		)
+		(property "Datasheet" "~"
+			(at 100.33 144.78 0)
+			(effects
+				(font
+					(size 1.27 1.27)
+				)
+				(hide yes)
+			)
+		)
+		(property "Description" "Special symbol for telling ERC where power comes from"
+			(at 100.33 144.78 0)
+			(effects
+				(font
+					(size 1.27 1.27)
+				)
+				(hide yes)
+			)
+		)
+		(pin "1"
+		)
+		(instances
+			(project "GBSCSI2_2.5SCA_TH_235x"
+				(path "/93ed3756-682c-4bf3-aa83-42c6b59d82c2/e68c1f1b-455b-4aa0-aecf-801739b3b8ff"
+					(reference "#FLG07")
+					(unit 1)
+				)
