File: EDA/Common Sheets/termination_wide.kicad_sch (KiCad schematic)
At the start: 54 parts, among them Q1 AO3401A, Q10 AO3401A, Q11 AO3401A, Q12 AO3401A, Q13 AO3401A, Q14 AO3401A, Q15 AO3401A, Q16 AO3401A, Q17 AO3401A, Q18 AO3401A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

Commit message: Fixing up schematics for SCA before layout
Other:
- title: GBSCSI2 Common Platform - Termination, Narrow -> GBSCSI2 Common Platform - Termination, Wide
