File: EDA/Common Sheets/buffers_wide.kicad_sch (KiCad schematic)
At the start: 17 parts, among them U12 74LVTH245, U13 74LVCH2T45, U4 74LVTH245, U5 74LVTH245, U6 74LVTH125, U7 74LVTH125

Commit message: Fixing up schematics for SCA before layout
Other:
- title: GBSCSI2 - Common Platform - Buffers, Narrow -> GBSCSI2 - Common Platform - Buffers, Wide
Changed lines of the file:
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@@
 	(paper "A4")
 	(title_block
-		(title "GBSCSI2 - Common Platform - Buffers, Narrow")
+		(title "GBSCSI2 - Common Platform - Buffers, Wide")
 		(date "2026-02-01")
 		(rev "2.0")

Commit message: SCA variant mostly laid out
Or rather, a first pass.
Connections:
- net +3.3V is gone; now on net +2.8V: C22.1, C23.1, C25.1, C26.1, C41.1, U12.20 (VCC), U4.20 (VCC), U5.20 (VCC), U6.14 (VCC), U7.14 (VCC)
- net GND: now also U7.1, U7.10, U7.12, U7.5; no longer U6.1, U6.5, U7.2, U7.4
- net ~{MCU_RST_IN}: now also U6.6; no longer U7.11
- net ~{MCU_RST_OUT}: now also U6.1; no longer U7.10
- net ~{MCU_SD0}: now also U4.2 (A0); no longer U4.9 (A7)
- net ~{MCU_SD1}: now also U4.3 (A1); no longer U4.8 (A6)
- net ~{MCU_SD2}: now also U4.4 (A2); no longer U4.7 (A5)
- net ~{MCU_SD3}: now also U4.5 (A3); no longer U4.6 (A4)
- net ~{MCU_SD4}: now also U4.6 (A4); no longer U4.5 (A3)
- net ~{MCU_SD5}: now also U4.7 (A5); no longer U4.4 (A2)
- net ~{MCU_SD6}: now also U4.8 (A6); no longer U4.3 (A1)
- net ~{MCU_SD7}: now also U4.9 (A7); no longer U4.2 (A0)
- net ~{MCU_SEL_OUT}: now also U7.4; no longer U7.1
- net ~{SCSI_RST}: now also U6.3, U6.5; no longer U7.12, U7.8
- net ~{SCSI_SD0}: now also U4.18 (B0); no longer U4.11 (B7)
- net ~{SCSI_SD1}: now also U4.17 (B1); no longer U4.12 (B6)
- net ~{SCSI_SD2}: now also U4.16 (B2); no longer U4.13 (B5)
- net ~{SCSI_SD3}: now also U4.15 (B3); no longer U4.14 (B4)
- net ~{SCSI_SD4}: now also U4.14 (B4); no longer U4.15 (B3)
- net ~{SCSI_SD5}: now also U4.13 (B5); no longer U4.16 (B2)
- net ~{SCSI_SD6}: now also U4.12 (B6); no longer U4.17 (B1)
- net ~{SCSI_SD7}: now also U4.11 (B7); no longer U4.18 (B0)
- net ~{SCSI_SEL}: now also U7.2, U7.6; no longer U7.3, U7.5
- net at R28.2: now also U7.3; no longer U7.6
Other:
- moved on the sheet: U6A, U6B, U7A, U7B, U7C, U7D
