File: EDA/Common Sheets/rp2350b_decoupling.kicad_sch (KiCad schematic)
At the start: 11 parts

Commit message: Started work on thru-hole SCA wide variant
Parts:
- added C36: 100nF, Capacitor_SMD:C_0402_1005Metric, symbol Device:C_Small
Connections:
- net +3.3V: now also C36.1
- net GND: now also C36.2
Changed lines of the file:
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@@
+	)
+	(junction
+		(at 99.06 114.3)
+		(diameter 0)
+		(color 0 0 0 0)
 	)
 	(junction
@@
 	)
 	(junction
+		(at 90.17 125.73)
+		(diameter 0)
+		(color 0 0 0 0)
+	)
+	(junction
 		(at 99.06 57.15)
 		(diameter 0)
@@
 	(wire
 		(pts
+			(xy 88.9 125.73) (xy 90.17 125.73)
+		)
+		(stroke
+			(width 0)
+			(type default)
+		)
+	)
+	(wire
+		(pts
 			(xy 99.06 43.18) (xy 99.06 45.72)
 		)
@@
 	(wire
 		(pts
+			(xy 99.06 114.3) (xy 99.06 125.73)
+		)
+		(stroke
+			(width 0)
+			(type default)
+		)
+	)
+	(wire
+		(pts
 			(xy 97.79 114.3) (xy 99.06 114.3)
 		)
@@
 	(wire
 		(pts
+			(xy 88.9 125.73) (xy 88.9 135.89)
+		)
+		(stroke
+			(width 0)
+			(type default)
+		)
+	)
+	(wire
+		(pts
+			(xy 97.79 125.73) (xy 99.06 125.73)
+		)
+		(stroke
+			(width 0)
+			(type default)
+		)
+	)
+	(wire
+		(pts
 			(xy 54.61 50.8) (xy 54.61 52.07)
 		)
@@
 	(wire
 		(pts
-			(xy 90.17 114.3) (xy 90.17 129.54)
+			(xy 90.17 114.3) (xy 90.17 125.73)
 		)
 		(stroke
@@
 		(pts
 			(xy 99.06 45.72) (xy 99.06 57.15)
+		)
+		(stroke
+			(width 0)
+			(type default)
+		)
+	)
+	(wire
+		(pts
+			(xy 90.17 125.73) (xy 92.71 125.73)
 		)
 		(stroke
@@
 	)
 	(symbol
+		(lib_id "Device:C_Small")
+		(at 95.25 125.73 270)
+		(unit 1)
+		(exclude_from_sim no)
+		(in_bom yes)
+		(on_board yes)
+		(dnp no)
+		(property "Reference" "C36"
+			(at 91.694 128.778 90)
+			(effects
+				(font
+					(size 1.2 1.2)
+				)
+				(justify left)
+			)
+		)
+		(property "Value" "100nF"
+			(at 91.694 131.0894 90)
+			(effects
+				(font
+					(size 1.27 1.27)
+				)
+				(justify left)
+			)
+		)
+		(property "Footprint" "Capacitor_SMD:C_0402_1005Metric"
+			(at 91.44 126.6952 0)
+			(effects
+				(font
+					(size 1.27 1.27)
+				)
+				(hide yes)
+			)
+		)
+		(property "Datasheet" "~"
+			(at 95.25 125.73 0)
+			(effects
+				(font
+					(size 1.27 1.27)
+				)
+				(hide yes)
+			)
+		)
+		(property "Description" ""
+			(at 95.25 125.73 0)
+			(effects
+				(font
+					(size 1.27 1.27)
+				)
+			)
+		)
+		(property "LCSC" "C307331"
+			(at 95.25 125.73 0)
+			(effects
+				(font
+					(size 1.27 1.27)
+				)
+				(hide yes)
+			)
+		)
+		(property "Preferred MPN" "CL05B104KB54PNC"
+			(at 95.25 125.73 90)
+			(effects
+				(font
+					(size 1.27 1.27)
+				)
+				(hide yes)
+			)
+		)
+		(property "Alternate Part Number" "GRM155R71H104KE14D"
+			(at 95.25 125.73 90)
+			(effects
+				(font
+					(size 1.27 1.27)
+				)
+				(hide yes)
+			)
+		)
+		(property "Nominal Preferred Characteristics" "50V X7R"
+			(at 94.742 133.096 90)
+			(effects
+				(font
+					(size 1.27 1.27)
+				)
+			)
+		)
+		(property "Case/Package" "0402"
+			(at 95.25 125.73 90)
+			(effects
+				(font
+					(size 1.27 1.27)
+				)
+				(hide yes)
+			)
+		)
+		(property "Dimensions" "1.0x0.5mm"
+			(at 95.25 125.73 90)
+			(effects
+				(font
+					(size 1.27 1.27)
+				)
+				(hide yes)
+			)
+		)
+		(pin "1"
+		)
+		(pin "2"
+		)
+		(instances
+			(project "GBSCSI2_2.5SCA_TH_235x"
+				(path "/93ed3756-682c-4bf3-aa83-42c6b59d82c2/871f9ffd-aa9f-4db2-af7f-735335bcb730/dbcf004f-88e5-4126-8d06-f1825ffeac66"
+					(reference "C36")
+					(unit 1)
+				)
+			)
+		)
+	)
+	(symbol
 		(lib_id "power:GND")
-		(at 90.17 129.54 0)
+		(at 88.9 135.89 0)
 		(unit 1)
 		(exclude_from_sim no)
@@
 		(dnp no)
 		(property "Reference" "#PWR040"
-			(at 90.17 135.89 0)
+			(at 88.9 142.24 0)
 			(effects
 				(font
@@
 		)
 		(property "Value" "GND"
-			(at 90.297 133.9342 0)
+			(at 89.027 140.2842 0)
 			(effects
 				(font
@@
 		)
 		(property "Footprint" ""
-			(at 90.17 129.54 0)
+			(at 88.9 135.89 0)
 			(effects
 				(font
@@
 		)
 		(property "Datasheet" ""
-			(at 90.17 129.54 0)
+			(at 88.9 135.89 0)
 			(effects
 				(font
@@
 		)
 		(property "Description" ""
-			(at 90.17 129.54 0)
-			(effects
-				(font
+			(at 88.9 135.89 0)
+			(effects
+				(font

Commit message: Prettifying models
Parts:
- added C43: 100nF, Capacitor_SMD:C_0402_1005Metric, symbol Device:C_Small
Connections:
- net +3.3V: now also C43.1
- net GND: now also C43.2
Changed lines of the file:
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@@
+	)
+	(junction
+		(at 99.06 125.73)
+		(diameter 0)
+		(color 0 0 0 0)
 	)
 	(junction
@@
 	)
 	(junction
+		(at 90.17 137.16)
+		(diameter 0)
+		(color 0 0 0 0)
+	)
+	(junction
 		(at 54.61 52.07)
 		(diameter 0)
@@
 	(wire
 		(pts
-			(xy 88.9 125.73) (xy 90.17 125.73)
-		)
-		(stroke
-			(width 0)
-			(type default)
-		)
-	)
-	(wire
-		(pts
 			(xy 99.06 43.18) (xy 99.06 45.72)
 		)
@@
 	(wire
 		(pts
+			(xy 90.17 137.16) (xy 90.17 146.05)
+		)
+		(stroke
+			(width 0)
+			(type default)
+		)
+	)
+	(wire
+		(pts
 			(xy 54.61 45.72) (xy 54.61 44.45)
 		)
@@
 	(wire
 		(pts
+			(xy 97.79 137.16) (xy 99.06 137.16)
+		)
+		(stroke
+			(width 0)
+			(type default)
+		)
+	)
+	(wire
+		(pts
 			(xy 92.71 45.72) (xy 90.17 45.72)
 		)
@@
 	(wire
 		(pts
+			(xy 90.17 137.16) (xy 92.71 137.16)
+		)
+		(stroke
+			(width 0)
+			(type default)
+		)
+	)
+	(wire
+		(pts
 			(xy 97.79 80.01) (xy 99.06 80.01)
 		)
@@
 	(wire
 		(pts
+			(xy 99.06 125.73) (xy 99.06 137.16)
+		)
+		(stroke
+			(width 0)
+			(type default)
+		)
+	)
+	(wire
+		(pts
 			(xy 97.79 102.87) (xy 99.06 102.87)
 		)
@@
 	(wire
 		(pts
-			(xy 88.9 125.73) (xy 88.9 135.89)
+			(xy 90.17 125.73) (xy 90.17 137.16)
 		)
 		(stroke
@@
 	(symbol
 		(lib_id "power:GND")
-		(at 88.9 135.89 0)
+		(at 90.17 146.05 0)
 		(unit 1)
 		(exclude_from_sim no)
@@
 		(dnp no)
 		(property "Reference" "#PWR040"
-			(at 88.9 142.24 0)
+			(at 90.17 152.4 0)
 			(effects
 				(font
@@
 		)
 		(property "Value" "GND"
-			(at 89.027 140.2842 0)
+			(at 90.297 150.4442 0)
 			(effects
 				(font
@@
 		)
 		(property "Footprint" ""
-			(at 88.9 135.89 0)
+			(at 90.17 146.05 0)
 			(effects
 				(font
@@
 		)
 		(property "Datasheet" ""
-			(at 88.9 135.89 0)
+			(at 90.17 146.05 0)
 			(effects
 				(font
@@
 		)
 		(property "Description" ""
-			(at 88.9 135.89 0)
+			(at 90.17 146.05 0)
 			(effects
 				(font
@@
 					(unit 1)
 				)
+			)
+		)
+	)
+	(symbol
+		(lib_id "Device:C_Small")
+		(at 95.25 137.16 270)
+		(unit 1)
+		(exclude_from_sim no)
+		(in_bom yes)
+		(on_board yes)
+		(dnp no)
+		(property "Reference" "C43"
+			(at 91.694 140.208 90)
+			(effects
+				(font
+					(size 1.2 1.2)
+				)
+				(justify left)
+			)
+		)
+		(property "Value" "100nF"
+			(at 91.694 142.5194 90)
+			(effects
+				(font
+					(size 1.27 1.27)
+				)
+				(justify left)
+			)
+		)
+		(property "Footprint" "Capacitor_SMD:C_0402_1005Metric"
+			(at 91.44 138.1252 0)
+			(effects
+				(font
+					(size 1.27 1.27)
+				)
+				(hide yes)
+			)
+		)
+		(property "Datasheet" "~"
+			(at 95.25 137.16 0)
+			(effects
+				(font
+					(size 1.27 1.27)
+				)
+				(hide yes)
+			)
+		)
+		(property "Description" ""
+			(at 95.25 137.16 0)
+			(effects
+				(font
+					(size 1.27 1.27)
+				)
+			)
+		)
+		(property "LCSC" "C307331"
+			(at 95.25 137.16 0)
+			(effects
+				(font
+					(size 1.27 1.27)
+				)
+				(hide yes)
+			)
+		)
+		(property "Preferred MPN" "CL05B104KB54PNC"
+			(at 95.25 137.16 90)
+			(effects
+				(font
+					(size 1.27 1.27)
+				)
+				(hide yes)
+			)
+		)
+		(property "Alternate Part Number" "GRM155R71H104KE14D"
+			(at 95.25 137.16 90)
+			(effects
+				(font
+					(size 1.27 1.27)
+				)
+				(hide yes)
+			)
+		)
+		(property "Nominal Preferred Characteristics" "50V X7R"
+			(at 94.742 144.526 90)
+			(effects
+				(font
+					(size 1.27 1.27)
+				)
+			)
+		)
+		(property "Case/Package" "0402"
+			(at 95.25 137.16 90)
+			(effects
+				(font
+					(size 1.27 1.27)
+				)
+				(hide yes)
+			)
+		)
+		(property "Dimensions" "1.0x0.5mm"
+			(at 95.25 137.16 90)
+			(effects
+				(font
+					(size 1.27 1.27)
+				)
+				(hide yes)
+			)
+		)
+		(pin "1"
+		)
+		(pin "2"
+		)
+		(instances
+			(project "GBSCSI2_2.5SCA_TH_235x"
+				(path "/93ed3756-682c-4bf3-aa83-42c6b59d82c2/871f9ffd-aa9f-4db2-af7f-735335bcb730/dbcf004f-88e5-4126-8d06-f1825ffeac66"
+					(reference "C43")
+					(unit 1)
+				)
