File: EDA/Common Sheets/core_235xA_narrow.kicad_sch (KiCad schematic)
At the start: 32 parts, among them J4 SM03B-SRSS-TB, J4.1 Conn_01x04, J6 Conn_01x02, SW1 SW_DIP_x04, U1 RP2350_60QFN, U2 W25Q128JVS, Y1 12MHz

Commit message: Prettifying models
Parts:
- U1: footprint Package_DFN_QFN:QFN-60-1EP_7x7mm_P0.4mm_EP3.4x3.4mm_ThermalVias -> GBSCSI:RP2350-QFN-60-1EP_7x7_P0.4mm_EP3.4x3.4mm_ThermalVias
Changed lines of the file:
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@@
 			)
 		)
-		(property "Footprint" "Package_DFN_QFN:QFN-60-1EP_7x7mm_P0.4mm_EP3.4x3.4mm_ThermalVias"
+		(property "Footprint" "GBSCSI:RP2350-QFN-60-1EP_7x7_P0.4mm_EP3.4x3.4mm_ThermalVias"
 			(at 93.98 80.01 0)
 			(effects

Commit message: Resuming work
Parts:
- C2, C3: value 22pF -> 15pF; LCSC C1555 -> C1548; Preferred MPN 0402CG220J500NT -> 0402CG150J500NT
- U1: value RP2350_60QFN -> RP235x_60QFN; LCSC C42411118 -> C41378174
- U2: now not fitted
- Y1: Alternate Part Number TX322512M4LBCE2T -> TAXM12M4RLBDDT2T; LCSC C133334 -> C20625731; Nominal Preferred Characteristics Cl=20pF - adjustments change C2/C3, ESR=50Ω -> Cl=10pF - adjustments change C2/C3, ESR=50Ω; Preferred MPN TAXM12M4RLBDDT2T -> ABM8-272-T3
Other:
- note added: "Alternate MPN x'tal and caps spec'd for Cl=20pF (C2/C3=22pF)"
- moved on the sheet: R10, R11, R12, R13, R14, R5, R6, R8, R9, SW1

Commit message: Minor tweaks
Parts:
- U2: footprint Package_SO:SOIC-8_5.23x5.23mm_P1.27mm -> Package_SO:SOIC-8_5.3x5.3mm_P1.27mm
Changed lines of the file:
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@@
 			)
 		)
-		(property "Footprint" "Package_SO:SOIC-8_5.23x5.23mm_P1.27mm"
+		(property "Footprint" "Package_SO:SOIC-8_5.3x5.3mm_P1.27mm"
 			(at 59.69 180.34 0)
 			(effects
