File: EDA/2.5_235x_wide_SCA_TH/GBSCSI2_2.5SCA_TH_235x.kicad_sch (KiCad schematic)
At the start: 4 parts

Commit message: Fixing up schematics for SCA before layout
Parts:
- added J7: Conn_01x05, symbol Connector_Generic:Conn_01x05
- added R68, R69, R70: 4.7kΩ, Resistor_SMD:R_0402_1005Metric, symbol Device:R_Small
Connections:
- new net +3.3V: J7.1 (Pin_1), R68.2, R69.2
- new net Core Logic, Basic Controls/I²C_INT: R70.2
- new net Core Logic, Basic Controls/I²C_SCL: J7.3 (Pin_3), R69.1
- new net Core Logic, Basic Controls/I²C_SDA: J7.2 (Pin_2), R68.1
- new net GND: J7.4 (Pin_4), R70.1
- no-connect marks 0 -> 1
Other:
- sheet Core Logic, Basic Controls ports: added I²C_INT, I²C_SCL, I²C_SDA; removed ~{CONN_TYPE}
- sheet Power: file ../Common Sheets/power_VTT_buck.kicad_sch -> ../Common Sheets/power_SCA.kicad_sch

Commit message: Prettifying models
Parts:
- J7: footprint (none) -> Connector_PinSocket_2.54mm:PinSocket_1x05_P2.54mm_Vertical
Changed lines of the file:
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@@
 			)
 		)
-		(property "Footprint" ""
+		(property "Footprint" "Connector_PinSocket_2.54mm:PinSocket_1x05_P2.54mm_Vertical"
 			(at 66.04 153.67 0)
 			(effects
