File: EDA/2.5_235x_narrow/GBSCSI2_2.5N_235x.kicad_pcb (KiCad board)
At the start: 4 copper layers, 69.5 x 93.5 mm, 146 parts, among them J1 SCSI_50-2P_2mm, J1.1 SCSI_50P_2.54mm, J2 TF003, J3 GCT-4105, J4 SM03B-SRSS-TB, J4.1 Conn_01x04, J5 Conn_01x04, J6 Conn_01x02, Q1 AO3401A, Q10 AO3401A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

Commit message: Minor tweaks
Parts:
- U2: footprint Package_SO:SOIC-8_5.23x5.23mm_P1.27mm -> Package_SO:SOIC-8_5.3x5.3mm_P1.27mm
